File: Kicad/resistor/resistor.kicad_pcb (KiCad board)
At the start: 2 copper layers, 100 x 35 mm, 146 parts, among them K1 R

Commit message: Update Resistor Board
Other:
- board text added: "Resistor Board"
- board text added: "Resistor Board - Rev.A - (01/2022) - Scale 100%"
- board text removed: "Resistance Board"
- board text removed: "Resistance Board - Rev.A - (01/2022) - Scale 100%"
Changed lines of the file:
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@@
   (paper "A4")
   (title_block
-    (title "Resistance Board")
+    (title "Resistor Board")
     (date "01/2022")
     (rev "A")
@@
     (effects (font (size 1.3 1.3) (thickness 0.2)) (justify right mirror))
   )
-  (gr_text "Resistance Board" (at 106.5 67.5) (layer "B.SilkS")
+  (gr_text "Resistor Board" (at 106.5 67.5) (layer "B.SilkS")
     (effects (font (size 1.3 1.3) (thickness 0.2)) (justify right mirror))
   )
@@
     (effects (font (size 1 1) (thickness 0.15)))
   )
-  (gr_text "Resistance Board" (at 193.5 67.5) (layer "F.SilkS")
+  (gr_text "Resistor Board" (at 193.5 67.5) (layer "F.SilkS")
     (effects (font (size 1.5 1.5) (thickness 0.2)) (justify right))
   )
@@
     (effects (font (size 1 1) (thickness 0.15)))
   )
-  (gr_text "Resistance Board - Rev.A - (01/2022) - Scale 100%" (at 100 120) (layer "Dwgs.User")
+  (gr_text "Resistor Board - Rev.A - (01/2022) - Scale 100%" (at 100 120) (layer "Dwgs.User")
     (effects (font (size 1.5 1.5) (thickness 0.2)) (justify left))
   )

Commit message: Update Resistor
Parts:
- removed H10, H11, H8, H9: KEYSTONE-9056, tronixio:KEYSTONE-9056
- removed H5, H6, H7: HARWIN-JUMPER-0254-14MM-BLACK, tronixio:HARWIN-M20-7680-7683
- added JP71: HARWIN-JUMPER-0254-14MM-BLACK, tronixio:HARWIN-M20-7680-7683, F.Cu at (173.0, 115.0)
- added JP72: HARWIN-JUMPER-0254-14MM-BLACK, tronixio:HARWIN-M20-7680-7683, F.Cu at (167.0, 115.0)
- added JP73: HARWIN-JUMPER-0254-14MM-BLACK, tronixio:HARWIN-M20-7680-7683, F.Cu at (197.0, 115.0)
- added JP74: HARWIN-JUMPER-0254-14MM-BLACK, tronixio:HARWIN-M20-7680-7683, F.Cu at (185.0, 115.0)
- added JP75: HARWIN-JUMPER-0254-14MM-BLACK, tronixio:HARWIN-M20-7680-7683, F.Cu at (191.0, 115.0)
- added JP76: HARWIN-JUMPER-0254-14MM-BLACK, tronixio:HARWIN-M20-7680-7683, F.Cu at (179.0, 115.0)
- added JP77: HARWIN-JUMPER-0254-14MM-BLACK, tronixio:HARWIN-M20-7680-7683, F.Cu at (161.0, 115.0)
- H1, H2, H3, H4: value HARWIN-JUMPER-0254-14MM-BLACK -> KEYSTONE-9056; footprint tronixio:HARWIN-M20-7680-7683 -> tronixio:KEYSTONE-9056
- moved H4 89.3 mm to (103.0, 68.0)
- moved H1 59.6 mm to (103.0, 97.0)
- moved H3 53.3 mm to (197.0, 68.0)
- moved H2 35.9 mm to (197.0, 97.0)

Commit message: Update
Parts:
- R1, R10, R11, R12, R13, R14, R15, R16, R17, R18, R19, R2, R20, R21, R22, R23, R24, R25, R26, R27, R28, R29, R3, R30, R31, R32, R33, R34, R35, R36, R37, R38, R39, R4, R40, R41, R42, R43, R44, R45, R46, R47, R48, R49, R5, R50, R51, R52, R53, R54, R55, R56, R57, R58, R59, R6, R60, R61, R62, R63, R7, R8, R9: footprint tronixio:RESISTOR-1206 -> tronixio:RESISTOR-SMD-1206

Commit message: Up
Parts:
- moved JP71 1.00 mm to (173.0, 116.0)
- moved JP72 1.00 mm to (167.0, 116.0)
- moved JP73 1.00 mm to (197.0, 116.0)
- moved JP74 1.00 mm to (185.0, 116.0)
- moved JP75 1.00 mm to (191.0, 116.0)
- moved JP76 1.00 mm to (179.0, 116.0)
- moved JP77 1.00 mm to (161.0, 116.0)
Routing:
- net Net-(JP1-Pad1): track 124.2 -> 125.0 mm
