File: Kicad/capacitors/capacitors.kicad_sch (KiCad schematic)
At the start: 141 parts, among them K1 Capacitor

Commit message: Update capacitors
Parts:
- JP1, JP10, JP11, JP12, JP13, JP14, JP15, JP16, JP17, JP18, JP19, JP2, JP20, JP21, JP22, JP23, JP24, JP25, JP26, JP27, JP28, JP29, JP3, JP30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: value HARWIN-254-M-1X02-JUMPER-VERTICAL -> ~
