File: Kicad/capacitors/main.kicad_sch (KiCad schematic)
At the start: 141 parts, among them K1 Capacitor

Commit message: Update
Parts:
- removed C56, C57, C58, C59, C60, C61, C62, C63: 10p, tronixio:CAPACITOR-SMD-1206, symbol tronixio:CAPACITOR-1206-10P-50V-5P-COG
- added C56, C57, C58, C59, C60, C61, C62, C63: 10p, tronixio:CAPACITOR-SMD-1206, symbol tronixio:CAPACITOR-1206-10P-100V-1P-COG
- C55: symbol tronixio:CAPACITOR-1206-10P-50V-5P-COG -> tronixio:CAPACITOR-1206-10P-100V-1P-COG; Mouser 80-C1206C100J5G -> 581-12061A100FAT2A; Tolerance 5% -> 1%; Voltage 50V -> 100V
Connections:
- net at C1.2, C10.2, C11.2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: now also C56.2, C57.2, C58.2, C59.2, C60.2, C61.2, C62.2, C63.2
- net at JP63.2: now also C63.1
- net at JP59.2: now also C59.1
- net at JP58.2: now also C58.1
- net at JP62.2: now also C62.1
- net at JP60.2: now also C60.1
- net at JP61.2: now also C61.1
- net at JP57.2: now also C57.1
- net at JP56.2: now also C56.1

Commit message: Up
Parts:
- removed C29, C30, C31, C32, C33, C34, C35, C36: 10n, tronixio:CAPACITOR-SMD-1206, symbol tronixio:CAPACITOR-1206-10N-50V-5P-X7R
- removed C38, C39, C40, C41, C42, C43, C44, C45: 1n, tronixio:CAPACITOR-SMD-1206, symbol tronixio:CAPACITOR-1206-1N-50V-5P-X7R
- removed C47, C48, C49, C50, C51, C52, C53, C54: 100p, tronixio:CAPACITOR-SMD-1206, symbol tronixio:CAPACITOR-1206-100P-50V-5P-COG
- added C29, C30, C31, C32, C33, C34, C35, C36: 10n, tronixio:CAPACITOR-SMD-1206, symbol tronixio:CAPACITOR-1206-10N-50V-1P-COG
- added C38, C39, C40, C41, C42, C43, C44, C45: 1n, tronixio:CAPACITOR-SMD-1206, symbol tronixio:CAPACITOR-1206-1N-50V-1P-COG
- added C47, C48, C49, C50, C51, C52, C53, C54: 100p, tronixio:CAPACITOR-SMD-1206, symbol tronixio:CAPACITOR-1206-100P-50V-1P-COG
- C28: symbol tronixio:CAPACITOR-1206-10N-50V-5P-X7R -> tronixio:CAPACITOR-1206-10N-50V-1P-COG; Mouser 80-C1206C103J5R -> 80-C1206C103F5GECTU; Tolerance 5% -> 1%
- C37: symbol tronixio:CAPACITOR-1206-1N-50V-5P-X7R -> tronixio:CAPACITOR-1206-1N-50V-1P-COG; Mouser C1206C102J5R -> 81-GRM3195C1H223FA1; Tolerance 5% -> 1%
- C46: symbol tronixio:CAPACITOR-1206-100P-50V-5P-COG -> tronixio:CAPACITOR-1206-100P-50V-1P-COG; Mouser 80-C1206C101J5G -> 80-C1206C101F5G; Tolerance 5% -> 1%
Connections:
- net at C1.2, C10.2, C11.2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: now also C29.2, C30.2, C31.2, C32.2, C33.2, C34.2, C35.2, C36.2, C38.2, C39.2, C40.2, C41.2, C42.2, C43.2, C44.2, C45.2, C47.2, C48.2, C49.2, C50.2, C51.2, C52.2, C53.2, C54.2
- net at JP51.2: now also C51.1
- net at JP48.2: now also C48.1
- net at JP31.2: now also C31.1
- net at JP41.2: now also C41.1
- net at JP40.2: now also C40.1
- net at JP36.2: now also C36.1
- net at JP29.2: now also C29.1
- net at JP44.2: now also C44.1
- net at JP32.2: now also C32.1
- net at JP49.2: now also C49.1
- net at JP34.2: now also C34.1
- net at JP38.2: now also C38.1
- net at JP45.2: now also C45.1
- net at JP30.2: now also C30.1
- net at JP35.2: now also C35.1
- net at JP52.2: now also C52.1
- net at JP42.2: now also C42.1
- net at JP39.2: now also C39.1
- net at JP54.2: now also C54.1
- net at JP43.2: now also C43.1
- net at JP50.2: now also C50.1
- net at JP33.2: now also C33.1
- net at JP47.2: now also C47.1
- net at JP53.2: now also C53.1
Other:
- note added: "- 10µ are 25V, others 50V. - 10p to 10n COG Dielectric, others X7R Dielectric. - For schematic clarity headers are 1x02, for PCB use 2x09 headers (HARWIN: M20-9980945)."
- note removed: "10p & 100P COG Dielectric, others X7R Dielectric."
- note removed: "10µ are 25V, others 50V."
- note removed: "For schematic clarity headers are 1x02, for PCB use 2x09 headers (HARWIN: M20-9980945)."
