File: Kicad/resistors/resistors.kicad_sch (KiCad schematic)
At the start: 145 parts, among them K1 R

Commit message: Up resistors
Parts:
- JP1, JP10, JP11, JP12, JP13, JP14, JP15, JP16, JP17, JP18, JP19, JP2, JP20, JP21, JP22, JP23, JP24, JP25, JP26, JP27, JP28, JP29, JP3, JP30, JP31, JP32, JP33, JP34, JP35, JP36, JP37, JP38, JP39, JP4, JP40, JP41, JP42, JP43, JP44, JP45, JP46, JP47, JP48, JP49, JP5, JP50, JP51, JP52, JP53, JP54, JP55, JP56, JP57, JP58, JP59, JP6, JP60, JP61, JP62, JP63, JP64, JP65, JP66, JP67, JP68, JP69, JP7, JP70, JP8, JP9: value HARWIN-254-M-1X02-JUMPER-VERTICAL -> ~
- K1: Mouser 55-M20-9990245 -> 855-M20-999024; Name HARWIN-254-M-1X02-VERTICAL -> (none)
- R46, R47, R48, R49, R50, R51, R52, R53, R54: Mouser 603-RT1206FRE1310RL -> 603-RT1206FRE0710RL
Other:
- note added: "For schematic clarity headers are 1x02, for PCB use 2x10 headers (HARWIN: M20-9981045)."
- note removed: "For schematic clarity headers are 1x02, for PCB use 2x10 headers (MOUSER: 855-M20-9981045)."
- title: Resistor Board -> Resistors Board
