File: Kicad/resistors/main.kicad_sch (KiCad schematic)
At the start: 145 parts, among them K1 R

Commit message: Up
Other:
- note added: "- For schematic clarity headers are 1x02, for PCB use 2x10 headers (HARWIN: M20-9981045)."
- note removed: "For schematic clarity headers are 1x02, for PCB use 2x10 headers (HARWIN: M20-9981045)."
